File: tomtho_mk2.kicad_pcb (KiCad board)
At the start: 2 copper layers, 275.8 x 106.3 mm, 173 parts, among them J1 USB-C, J2 BATTERY, J3 TRACKPAD, Q1 AO3401A, SW1 SKRAAWE010, SW10 SKRAAWE010, SW11 SKRAAWE010, SW12 SKRAAWE010, SW13 SKRAAWE010, SW14 SKRAAWE010, SW15 SKRAAWE010, SW16 SKRAAWE010, SW17 SKRAAWE010, SW18 SKRAAWE010, SW19 SKRAAWE010, SW2 SKRAAWE010, SW20 SKRAAWE010, SW21 SKRAAWE010, SW22 SKRAAWE010, SW23 SKRAAWE010, SW24 SKRAAWE010, SW25 SKRAAWE010, SW26 SKRAAWE010, SW27 SKRAAWE010, SW28 SKRAAWE010, SW29 SKRAAWE010, SW3 SKRAAWE010, SW30 SKRAAWE010, SW31 SKRAAWE010, SW32 SKRAAWE010, SW33 SKRAAWE010, SW34 SKRAAWE010, SW35 SKRAAWE010, SW36 SKRAAWE010, SW37 SKRAAWE010, SW38 SKRAAWE010, SW39 SKRAAWE010, SW4 SKRAAWE010, SW40 SKRAAWE010, SW41 SKRAAWE010, SW42 SKRAAWE010, SW43 SKRAAWE010, SW44 SKRAAWE010, SW45 SKRAAWE010, SW46 SKRAAWE010, SW47 SKRAAWE010, SW48 SKRAAWE010, SW49 SKRAAWE010, SW5 SKRAAWE010, SW50 SKRAAWE010, SW51 SKRAAWE010, SW52 SKRAAWE010, SW53 SKRAAWE010, SW54 SKRAAWE010, SW55 SKRAAWE010, SW56 SKRAAWE010, SW57 SKRAAWE010, SW58 SKRAAWE010, SW59 SKRAAWE010, SW6 SKRAAWE010, SW60 SKRAAWE010, SW61 SKRAAWE010, SW62 SKRAAWE010, SW63 SKRAAWE010, SW64 SKRAAWE010, SW65 SKRAAWE010, SW66 RESET, SW67 POWER, SW7 SKRAAWE010, SW8 SKRAAWE010, SW9 SKRAAWE010, U1 MDBT50Q-1MV2, U2 USBLC6-2SC6, U3 MCP73831

Commit message: mk2: routed PCB (local KiCad 10 DRC: 0 violations, 0 unconnected, parity 0), JLC BOM/CPL, CI DRC + gerbers for mk2
Co-Authored-By: Claude Opus 5.5 <noreply@anthropic.com>
Claude-Session: https://claude.ai/code/session_014QKLhpB6tKWk1p8Y7v384p
Routing:
- net /ROW0: track 0.00 -> 429.3 mm, vias 0 -> 9
- net /ROW2: track 0.00 -> 397.4 mm, vias 0 -> 9
- net /ROW5: track 0.00 -> 389.2 mm, vias 0 -> 6
- net /ROW3: track 0.00 -> 386.5 mm, vias 0 -> 10
- net /ROW4: track 0.00 -> 366.5 mm
- net /ROW1: track 0.00 -> 351.5 mm, vias 0 -> 9
- net /VDD: track 0.00 -> 331.0 mm, vias 0 -> 5
- net /COL0: track 0.00 -> 254.9 mm, vias 0 -> 2
- net /COL11: track 0.00 -> 243.9 mm, vias 0 -> 2
- net /COL10: track 0.00 -> 228.5 mm, vias 0 -> 2
- net /VBUS: track 0.00 -> 222.9 mm, vias 0 -> 8
- net /COL1: track 0.00 -> 214.7 mm, vias 0 -> 2
- net /COL9: track 0.00 -> 201.2 mm, vias 0 -> 2
- net /COL2: track 0.00 -> 197.4 mm, vias 0 -> 2
- net /COL7: track 0.00 -> 196.1 mm, vias 0 -> 2
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
Commit message: mk2: trackpad board derived from GR-Trackpad65 (10Tx x 10Rx, 49x43, DRC clean); main board gets a trackpad cut-out, J3 beside it (DRC 0/0/0)
Co-Authored-By: Claude Opus 5.5 <noreply@anthropic.com>
Claude-Session: https://claude.ai/code/session_014QKLhpB6tKWk1p8Y7v384p
Parts:
- moved R12 40.5 mm to (111.1, 51.4)
- moved J3 29.7 mm to (111.4, 46.8), turned to 90 degrees
- moved R11 19.4 mm to (111.1, 42.2)
Connections:
- J3 pad 1: /VDD -> /TP_RDY
- J3 pad 2: GND -> /TP_RST
- J3 pad 3: /TP_SDA -> GND
- J3 pad 4: /TP_SCL -> /VDD
- J3 pad 5: /TP_RDY -> /TP_SCL
- J3 pad 6: /TP_RST -> /TP_SDA
Routing:
- net /ROW0: track 429.3 -> 350.2 mm
- net /TP_SCL: track 38.0 -> 81.3 mm
- net /USB_DN: track 36.8 -> 76.8 mm, vias 2 -> 6
- net /ROW2: track 397.4 -> 435.1 mm, vias 9 -> 12
- net /TP_RDY: track 33.8 -> 68.4 mm, vias 2 -> 4
- net /TP_RST: track 37.2 -> 68.9 mm, vias 4 -> 2
- net /ROW3: track 386.5 -> 416.3 mm, vias 10 -> 12
- net /TP_SDA: track 38.6 -> 68.2 mm, vias 2 -> 4
- net /ROW1: track 351.5 -> 378.9 mm, vias 9 -> 13
- net /ROW4: track 366.5 -> 389.1 mm
- net /COL5: track 163.5 -> 185.6 mm, vias 2 -> 4
- net /SWDIO: track 40.9 -> 62.1 mm
- net /VBUS: track 222.9 -> 201.7 mm, vias 8 -> 5
- net /RESET: track 13.2 -> 32.5 mm
- net /ROW5: track 389.2 -> 373.2 mm, vias 6 -> 7
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Other:
- outline, holes or cut-outs redrawn

Commit message: mk2: trackpad -> Azoteq TPS43-201A-S (43x40); cut-out 44x41, J3 pinout per TPS43 J1; keys unchanged; DRC 0/0/0
Co-Authored-By: Claude Opus 5.5 <noreply@anthropic.com>
Claude-Session: https://claude.ai/code/session_014QKLhpB6tKWk1p8Y7v384p
Parts:
- moved R11 2.80 mm to (113.9, 42.1)
- moved R12 2.80 mm to (113.9, 51.3)
- moved J3 2.80 mm to (114.2, 46.7)
Routing:
- net /ROW0: track 350.2 -> 401.9 mm, vias 9 -> 10
- net /ROW2: track 435.1 -> 386.3 mm, vias 12 -> 10
- net /USB_DN: track 76.8 -> 33.2 mm, vias 6 -> 2
- net /CHG_STAT: track 152.3 -> 194.6 mm, vias 2 -> 4
- net GND: track 196.7 -> 158.4 mm, vias 498 -> 1118
- net /VBUS: track 201.7 -> 231.2 mm
- net /COL5: track 185.6 -> 161.7 mm
- net /SWDIO: track 62.1 -> 41.3 mm
- net /RESET: track 32.5 -> 13.1 mm
- net /ROW5: track 373.2 -> 358.7 mm, vias 7 -> 6
- net /CC1: track 21.0 -> 33.4 mm, vias 2 -> 0
- net /CC2: track 21.1 -> 9.17 mm
- net /TP_SDA: track 68.2 -> 80.1 mm, vias 4 -> 2
- net /TP_RST: track 68.9 -> 57.9 mm
- net /USB_DP: track 40.2 -> 49.2 mm, vias 2 -> 6
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Other:
- outline, holes or cut-outs redrawn
- board text added: "nRF52840 MDBT50Q / TPS43 / ZMK / 18.5x18"
- board text removed: "nRF52840 MDBT50Q / IQS550 / ZMK / 18.5x18"

Commit message: mk2 board check: JLC CPL in Gerber coordinates with per-footprint rotation/origin offsets (verified pad-on-pad against LCSC footprints), charge current 210 mA, README notes (STAT, REGOUT0, battery polarity, MDBT50Q stock)
Co-Authored-By: Claude Opus 5.5 <noreply@anthropic.com>
Claude-Session: https://claude.ai/code/session_014QKLhpB6tKWk1p8Y7v384p
Parts:
- R3: value 10k -> 4.7k
Changed lines of the file:
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@@
 		(descr "Resistor 0603 (1608 metric)")
 		(property "Reference" "R3" (at 0 -1.45 0) (layer "F.SilkS") (effects (font (size 0.8 0.8) (thickness 0.12))))
-		(property "Value" "10k" (at 0 1.45 0) (layer "F.Fab") (effects (font (size 0.6 0.6) (thickness 0.09))))
+		(property "Value" "4.7k" (at 0 1.45 0) (layer "F.Fab") (effects (font (size 0.6 0.6) (thickness 0.09))))
 		(property "Footprint" "tomtho_mk2:R_0603" (at 0 0 0) (unlocked yes) (layer "F.Fab") (hide yes) (effects (font (size 1 1) (thickness 0.15))))
 		(property "Datasheet" "" (at 0 0 0) (unlocked yes) (layer "F.Fab") (hide yes) (effects (font (size 1 1) (thickness 0.15))))
-		(property "Description" "Ichg = 1000V/10k = 100mA" (at 0 0 0) (unlocked yes) (layer "F.Fab") (hide yes) (effects (font (size 1 1) (thickness 0.15))))
-		(property "LCSC" "C25804" (at 0 0 0) (unlocked yes) (layer "F.Fab") (hide yes) (effects (font (size 1 1) (thickness 0.15))))
-		(property "MPN" "0603WAF1002T5E" (at 0 0 0) (unlocked yes) (layer "F.Fab") (hide yes) (effects (font (size 1 1) (thickness 0.15))))
+		(property "Description" "Ichg = 1000V/4.7k = 213mA (0.2-0.5C for an 800-1000 mAh cell)" (at 0 0 0) (unlocked yes) (layer "F.Fab") (hide yes) (effects (font (size 1 1) (thickness 0.15))))
+		(property "LCSC" "C23162" (at 0 0 0) (unlocked yes) (layer "F.Fab") (hide yes) (effects (font (size 1 1) (thickness 0.15))))
+		(property "MPN" "0603WAF4701T5E" (at 0 0 0) (unlocked yes) (layer "F.Fab") (hide yes) (effects (font (size 1 1) (thickness 0.15))))
 		(sheetname "Root")
 		(sheetfile "tomtho_mk2.kicad_sch")

Commit message: mk2: case v1 (top frame + bottom plate + 0.5u x 0.5u flange cap) in CadQuery; PCB: 11 case screws in rear strip / front edge, arrow diodes and J3 moved clear of ACC keycap legs, USB D- bridge protected; DRC 0/0/0
Co-Authored-By: Claude Opus 5.5 <noreply@anthropic.com>
Claude-Session: https://claude.ai/code/session_014QKLhpB6tKWk1p8Y7v384p
Parts:
- added H10: M2, tomtho_mk2:MountingHole_2.2mm_M2, F.Cu at (180.0, 104.0)
- added H11: M2, tomtho_mk2:MountingHole_2.2mm_M2, F.Cu at (215.0, 102.5)
- added H6: M2, tomtho_mk2:MountingHole_2.2mm_M2, F.Cu at (240.0, 4.50)
- added H7: M2, tomtho_mk2:MountingHole_2.2mm_M2, F.Cu at (60.0, 102.5)
- added H8: M2, tomtho_mk2:MountingHole_2.2mm_M2, F.Cu at (100.0, 104.0)
- added H9: M2, tomtho_mk2:MountingHole_2.2mm_M2, F.Cu at (138.5, 100.5)
- moved H2 166.8 mm to (80.0, 4.50)
- moved H5 113.2 mm to (200.0, 4.50)
- moved H1 53.5 mm to (40.0, 4.50)
- moved D59 15.8 mm to (238.0, 89.9), turned to 0 degrees
- moved D65 15.8 mm to (238.0, 98.9), turned to 0 degrees
- moved R11 9.20 mm to (113.9, 51.3)
- moved J3 8.50 mm to (114.2, 55.2)
- moved R12 7.80 mm to (113.9, 59.1)
Routing:
- net /ROW1: track 374.8 -> 429.3 mm, vias 12 -> 10
- net /CHG_STAT: track 194.6 -> 151.1 mm, vias 4 -> 2
- net /ROW2: track 386.3 -> 428.3 mm, vias 10 -> 11
- net GND: track 158.4 -> 197.3 mm, vias 1118 -> 1122
- net /VBUS: track 231.2 -> 201.5 mm, vias 5 -> 4
- net /VDD: track 339.1 -> 364.3 mm, vias 6 -> 10
- net /USB_DN: track 33.2 -> 57.7 mm, vias 2 -> 3
- net /ROW5: track 358.7 -> 335.6 mm
- net /ROW3: track 411.8 -> 395.3 mm, vias 11 -> 9
- net /TP_RST: track 57.9 -> 72.4 mm
- net /SWDIO: track 41.3 -> 31.4 mm, vias 4 -> 0
- net /TP_RDY: track 61.0 -> 70.5 mm, vias 4 -> 2
- net /TP_SDA: track 80.1 -> 89.1 mm
- net /USB_DP: track 49.2 -> 57.7 mm, vias 6 -> 2
- net /ROW0: track 401.9 -> 394.8 mm, vias 10 -> 8
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
Commit message: mk2 v21: column stagger 0.75 x roBa, thumbs 1u / 1.25u (Space, Enter) / 1u at 1.1u pitch, L/M/R 2.5 mm under the trackpad; PCB re-placed and re-routed, DRC 0/0/0
Co-Authored-By: Claude Opus 5.5 <noreply@anthropic.com>
Claude-Session: https://claude.ai/code/session_014QKLhpB6tKWk1p8Y7v384p
Parts:
- moved D52 4.71 mm to (81.5, 96.6)
- moved D57 4.71 mm to (195.5, 96.6)
- moved SW52 4.71 mm to (81.5, 91.6)
- moved SW57 4.71 mm to (195.5, 91.6)
- moved SW56 3.52 mm to (172.8, 92.5)
- moved D53 3.52 mm to (103.8, 97.5)
- moved SW53 3.52 mm to (104.2, 92.5)
- moved D56 3.52 mm to (173.2, 97.5)
- moved D62 3.40 mm to (124.6, 79.3)
- moved D63 3.40 mm to (138.5, 79.3)
- moved D64 3.40 mm to (152.4, 79.3)
- moved SW62 3.40 mm to (124.6, 74.3)
- moved SW63 3.40 mm to (138.5, 74.3)
- moved SW64 3.40 mm to (152.4, 74.3)
- moved SW54 2.34 mm to (126.8, 95.1)
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Routing:
- net /RESET: track 17.6 -> 59.7 mm
- net /ROW1: track 429.3 -> 400.3 mm
- net /ROW5: track 335.6 -> 356.6 mm, vias 6 -> 7
- net /VBUS: track 201.5 -> 220.5 mm, vias 4 -> 6
- net /ROW0: track 394.8 -> 376.4 mm, vias 8 -> 11
- net /ROW3: track 395.3 -> 413.2 mm, vias 9 -> 11
- net /TP_SDA: track 89.1 -> 102.9 mm
- net /CC1: track 30.0 -> 43.3 mm
- net /TP_SCL: track 78.4 -> 90.6 mm
- net /SWDIO: track 31.4 -> 41.7 mm, vias 0 -> 2
- net GND: track 197.3 -> 187.3 mm, vias 1122 -> 1174
- net /VDD: track 364.3 -> 356.2 mm, vias 10 -> 8
- net /COL11: track 235.9 -> 243.3 mm
- net /COL5: track 168.3 -> 175.0 mm
- net /CC2: track 9.34 -> 15.5 mm
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Other:
- outline, holes or cut-outs redrawn

Commit message: mk2 PCB: tommys079 logo + 'Designed by tommys079' on the back silkscreen (DRC 0/0/0)
Co-Authored-By: Claude Opus 5.5 <noreply@anthropic.com>
Claude-Session: https://claude.ai/code/session_014QKLhpB6tKWk1p8Y7v384p
Other:
- board text added: "Designed by tommys079"

Commit message: mk2: named Ashiyu - back silkscreen title + ClickBoard credit (DRC 0/0/0)
Co-Authored-By: Claude Opus 5.5 <noreply@anthropic.com>
Claude-Session: https://claude.ai/code/session_014QKLhpB6tKWk1p8Y7v384p
Other:
- board text added: "Ashiyu"
- board text added: "Inspired by ClickBoard (Salicylic_acid3)"
- board text removed: "tomtho-slim mk2"
Changed lines of the file:
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@@
 	(gr_text "LiPo 1S  (<= 3.0 t x 40 x 70)" (at 57 54) (layer "B.SilkS") (effects (font (size 1.5 1.5) (thickness 0.225)) (justify mirror)))
 	(gr_text "lead -> slot -> J2 (pin1 = +)" (at 57 57.5) (layer "B.SilkS") (effects (font (size 1 1) (thickness 0.15)) (justify mirror)))
-	(gr_text "tomtho-slim mk2" (at 200 77) (layer "B.SilkS") (effects (font (size 2.5 2.5) (thickness 0.375)) (justify mirror)))
-	(gr_text "Designed by tommys079" (at 200 81) (layer "B.SilkS") (effects (font (size 1.5 1.5) (thickness 0.225)) (justify mirror)))
-	(gr_text "nRF52840 MDBT50Q / TPS43 / ZMK / 18.5x18" (at 200 84.5) (layer "B.SilkS") (effects (font (size 1.2 1.2) (thickness 0.18)) (justify mirror)))
-	(gr_text "JLCJLCJLCJLC" (at 200 87.5) (layer "B.SilkS") (effects (font (size 1 1) (thickness 0.15)) (justify mirror)))
+	(gr_text "Ashiyu" (at 200 77.5) (layer "B.SilkS") (effects (font (size 3 3) (thickness 0.45)) (justify mirror)))
+	(gr_text "Designed by tommys079" (at 200 81.5) (layer "B.SilkS") (effects (font (size 1.5 1.5) (thickness 0.225)) (justify mirror)))
+	(gr_text "Inspired by ClickBoard (Salicylic_acid3)" (at 200 84.3) (layer "B.SilkS") (effects (font (size 1 1) (thickness 0.15)) (justify mirror)))
+	(gr_text "nRF52840 MDBT50Q / TPS43 / ZMK / 18.5x18" (at 200 86.8) (layer "B.SilkS") (effects (font (size 1 1) (thickness 0.15)) (justify mirror)))
+	(gr_text "JLCJLCJLCJLC" (at 200 89.3) (layer "B.SilkS") (effects (font (size 1 1) (thickness 0.15)) (justify mirror)))
 	(gr_text "DIO CLK GND VDD" (at 138.2 25.9) (layer "F.SilkS") (effects (font (size 0.8 0.8) (thickness 0.12))))
 	(gr_text "ON   OFF" (at 155 7.4) (layer "F.SilkS") (effects (font (size 0.8 0.8) (thickness 0.12))))
