File: tomtho_mk2.kicad_pcb (KiCad board)
At the start: 2 copper layers, 275.8 x 106.3 mm, 179 parts, among them J1 USB-C, J2 BATTERY, J3 TRACKPAD, Q1 AO3401A, SW1 SKRAAWE010, SW10 SKRAAWE010, SW11 SKRAAWE010, SW12 SKRAAWE010, SW13 SKRAAWE010, SW14 SKRAAWE010, SW15 SKRAAWE010, SW16 SKRAAWE010, SW17 SKRAAWE010, SW18 SKRAAWE010, SW19 SKRAAWE010, SW2 SKRAAWE010, SW20 SKRAAWE010, SW21 SKRAAWE010, SW22 SKRAAWE010, SW23 SKRAAWE010, SW24 SKRAAWE010, SW25 SKRAAWE010, SW26 SKRAAWE010, SW27 SKRAAWE010, SW28 SKRAAWE010, SW29 SKRAAWE010, SW3 SKRAAWE010, SW30 SKRAAWE010, SW31 SKRAAWE010, SW32 SKRAAWE010, SW33 SKRAAWE010, SW34 SKRAAWE010, SW35 SKRAAWE010, SW36 SKRAAWE010, SW37 SKRAAWE010, SW38 SKRAAWE010, SW39 SKRAAWE010, SW4 SKRAAWE010, SW40 SKRAAWE010, SW41 SKRAAWE010, SW42 SKRAAWE010, SW43 SKRAAWE010, SW44 SKRAAWE010, SW45 SKRAAWE010, SW46 SKRAAWE010, SW47 SKRAAWE010, SW48 SKRAAWE010, SW49 SKRAAWE010, SW5 SKRAAWE010, SW50 SKRAAWE010, SW51 SKRAAWE010, SW52 SKRAAWE010, SW53 SKRAAWE010, SW54 SKRAAWE010, SW55 SKRAAWE010, SW56 SKRAAWE010, SW57 SKRAAWE010, SW58 SKRAAWE010, SW59 SKRAAWE010, SW6 SKRAAWE010, SW60 SKRAAWE010, SW61 SKRAAWE010, SW62 SKRAAWE010, SW63 SKRAAWE010, SW64 SKRAAWE010, SW65 SKRAAWE010, SW66 RESET, SW67 POWER, SW7 SKRAAWE010, SW8 SKRAAWE010, SW9 SKRAAWE010, U1 MDBT50Q-1MV2, U2 USBLC6-2SC6, U3 MCP73831

Commit message: Ashiyu PCB: drop the parts line and the JLC order-number marker from the back silkscreen (DRC 0/0/0)
Co-Authored-By: Claude Opus 5.5 <noreply@anthropic.com>
Claude-Session: https://claude.ai/code/session_014QKLhpB6tKWk1p8Y7v384p
Other:
- board text removed: "JLCJLCJLCJLC"
- board text removed: "nRF52840 MDBT50Q / TPS43 / ZMK / 18.5x18"
Changed lines of the file:
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@@
 	(gr_text "Designed by tommys079" (at 200 81.5) (layer "B.SilkS") (effects (font (size 1.5 1.5) (thickness 0.225)) (justify mirror)))
 	(gr_text "Inspired by ClickBoard (Salicylic_acid3)" (at 200 84.3) (layer "B.SilkS") (effects (font (size 1 1) (thickness 0.15)) (justify mirror)))
-	(gr_text "nRF52840 MDBT50Q / TPS43 / ZMK / 18.5x18" (at 200 86.8) (layer "B.SilkS") (effects (font (size 1 1) (thickness 0.15)) (justify mirror)))
-	(gr_text "JLCJLCJLCJLC" (at 200 89.3) (layer "B.SilkS") (effects (font (size 1 1) (thickness 0.15)) (justify mirror)))
 	(gr_text "DIO CLK GND VDD" (at 138.2 25.9) (layer "F.SilkS") (effects (font (size 0.8 0.8) (thickness 0.12))))
 	(gr_text "ON   OFF" (at 155 7.4) (layer "F.SilkS") (effects (font (size 0.8 0.8) (thickness 0.12))))

Commit message: Ashiyu PCB: JLC order-number marker moved under the LiPo (back side, hidden)
Co-Authored-By: Claude Opus 5.5 <noreply@anthropic.com>
Claude-Session: https://claude.ai/code/session_014QKLhpB6tKWk1p8Y7v384p
Other:
- board text added: "JLCJLCJLCJLC"
Changed lines of the file:
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@@
 	(gr_text "LiPo 1S  (<= 3.0 t x 40 x 70)" (at 57 54) (layer "B.SilkS") (effects (font (size 1.5 1.5) (thickness 0.225)) (justify mirror)))
 	(gr_text "lead -> slot -> J2 (pin1 = +)" (at 57 57.5) (layer "B.SilkS") (effects (font (size 1 1) (thickness 0.15)) (justify mirror)))
+	(gr_text "JLCJLCJLCJLC" (at 57 62) (layer "B.SilkS") (effects (font (size 1 1) (thickness 0.15)) (justify mirror)))
 	(gr_text "Ashiyu" (at 200 77.5) (layer "B.SilkS") (effects (font (size 3 3) (thickness 0.45)) (justify mirror)))
 	(gr_text "Designed by tommys079" (at 200 81.5) (layer "B.SilkS") (effects (font (size 1.5 1.5) (thickness 0.225)) (justify mirror)))
