File: tomtho_mk2.kicad_sch (KiCad schematic)
At the start: 176 parts, among them J1 USB-C, J2 BATTERY, J3 TRACKPAD, Q1 AO3401A, SW1 SKRAAWE010, SW10 SKRAAWE010, SW11 SKRAAWE010, SW12 SKRAAWE010, SW13 SKRAAWE010, SW14 SKRAAWE010, SW15 SKRAAWE010, SW16 SKRAAWE010, SW17 SKRAAWE010, SW18 SKRAAWE010, SW19 SKRAAWE010, SW2 SKRAAWE010, SW20 SKRAAWE010, SW21 SKRAAWE010, SW22 SKRAAWE010, SW23 SKRAAWE010, SW24 SKRAAWE010, SW25 SKRAAWE010, SW26 SKRAAWE010, SW27 SKRAAWE010, SW28 SKRAAWE010, SW29 SKRAAWE010, SW3 SKRAAWE010, SW30 SKRAAWE010, SW31 SKRAAWE010, SW32 SKRAAWE010, SW33 SKRAAWE010, SW34 SKRAAWE010, SW35 SKRAAWE010, SW36 SKRAAWE010, SW37 SKRAAWE010, SW38 SKRAAWE010, SW39 SKRAAWE010, SW4 SKRAAWE010, SW40 SKRAAWE010, SW41 SKRAAWE010, SW42 SKRAAWE010, SW43 SKRAAWE010, SW44 SKRAAWE010, SW45 SKRAAWE010, SW46 SKRAAWE010, SW47 SKRAAWE010, SW48 SKRAAWE010, SW49 SKRAAWE010, SW5 SKRAAWE010, SW50 SKRAAWE010, SW51 SKRAAWE010, SW52 SKRAAWE010, SW53 SKRAAWE010, SW54 SKRAAWE010, SW55 SKRAAWE010, SW56 SKRAAWE010, SW57 SKRAAWE010, SW58 SKRAAWE010, SW59 SKRAAWE010, SW6 SKRAAWE010, SW60 SKRAAWE010, SW61 SKRAAWE010, SW62 SKRAAWE010, SW63 SKRAAWE010, SW64 SKRAAWE010, SW65 SKRAAWE010, SW66 RESET, SW67 POWER, SW7 SKRAAWE010, SW8 SKRAAWE010, SW9 SKRAAWE010, U1 MDBT50Q-1MV2, U2 USBLC6-2SC6, U3 MCP73831

Commit message: Ashiyu v22: lower-left Ctrl 1u / Fn+Win 0.5u stacked / Alt 1u (66 keys, Win on ROW5 COL1); 9th Tadpole pin (front centre); trackpad without cover plate (module touched directly through a 41x38 window, 1.0x0.5 lip); 1.5 mm top chamfer; refs SW101/SW102/D101; re-routed (Freerouting 1.9, local check 0 errors); case CI reads case_inputs from the PCB via pcbnew; HANDOFF.md
Co-Authored-By: Claude Opus 5.5 <noreply@anthropic.com>
Claude-Session: https://claude.ai/code/session_01Rq3DZsqPhBbL1FAX1XrxAC
Parts:
- removed SW67: POWER, tomtho_mk2:SW_SPDT_PCM12, symbol tomtho_mk2:SW_SPDT
- added D101: B5819W, tomtho_mk2:D_SOD-123, symbol tomtho_mk2:D_Schottky
- added H9: Tadpole, tomtho_mk2:Tadpole_D3.0_NPTH, symbol tomtho_mk2:MountingHole
- added SW101: RESET, tomtho_mk2:SW_TS-1928-B, symbol tomtho_mk2:SW_Push
- added SW102: POWER, tomtho_mk2:SW_SPDT_PCM12, symbol tomtho_mk2:SW_SPDT
- D66: value B5819W -> 1N4148W; symbol tomtho_mk2:D_Schottky -> tomtho_mk2:D; LCSC C8598 -> C81598; MPN B5819W SL -> 1N4148W
- SW66: value RESET -> SKRAAWE010; footprint tomtho_mk2:SW_TS-1928-B -> tomtho_mk2:SW_ALPS_SKRA_6.2mm; LCSC C1121891 -> C202383; MPN TS-1928-B -> SKRAAWE010
Connections:
- net COL1: now also SW62.1
- net COL10: now also SW66.1; no longer SW65.1
- net COL5: now also SW63.1; no longer SW62.1
- net COL6: now also SW64.1; no longer SW63.1
- net COL7: now also SW65.1; no longer SW64.1
- net GND: now also SW101.2; no longer SW66.2
- net K5_10: now also D66.2 (A), SW66.2; no longer D65.2 (A), SW65.2
- net K5_5: now also D63.2 (A), SW63.2; no longer D62.2 (A), SW62.2
- net K5_6: now also D64.2 (A), SW64.2; no longer D63.2 (A), SW63.2
- net K5_7: now also D65.2 (A), SW65.2; no longer D64.2 (A), SW64.2
- net RESET: now also SW101.1; no longer SW66.1
- net ROW5: now also D66.1 (K)
- net VBUS: now also D101.2 (A); no longer D66.2 (A)
- net VDDH: now also SW102.1 (A)
- net VSYS: now also D101.1 (K), SW102.2 (C); no longer D66.1 (K)
- new net K5_1: D62.2 (A), SW62.2
Other:
- note added: "Alt"
- note added: "Key matrix 6 x 12 (66 keys, ALPS SKRA + 1N4148W, COL -> SW -> D -> ROW)"
- note added: "Load sharing (AN1149) USB -> D101, battery -> Q1 SW102: VSYS -> VDDH"
- note removed: "Key matrix 6 x 12 (65 keys, ALPS SKRA + 1N4148W, COL -> SW -> D -> ROW)"
- note removed: "Load sharing (AN1149) USB -> D66, battery -> Q1 SW67: VSYS -> VDDH"
- moved on the sheet: D62, D63, D64, D65, SW62, SW63, SW64, SW65, SW66
